File: PCB/Main/Main.kicad_sch (KiCad schematic)
At the start: 5 parts, among them J1 PICO LEFT, J2 PICO Right, J3 Screw_Terminal_01x02, J4 TB6612FNG_right, J5 TB6612FNG_left

Commit message: 3step file
Inserted 3step file of nema 17 42x42x23.
Parts:
- added J6: Conn_01x02_Socket, Connector_JST:JST_XH_B2B-XH-A_1x02_P2.50mm_Vertical, symbol Connector:Conn_01x02_Socket
- added J7: Conn_01x03_Socket, Connector_JST:JST_XH_B3B-XH-A_1x03_P2.50mm_Vertical, symbol Connector:Conn_01x03_Socket
- added J8: Conn_01x04_Socket, Connector_JST:JST_XH_B4B-XH-A_1x04_P2.50mm_Vertical, symbol Connector:Conn_01x04_Socket
Connections:
- net at J2.3 (Pin_3): now also J6.1 (Pin_1)
- net at J2.5 (Pin_5): now also J6.2 (Pin_2)
